File: logic-debug/logic-debug.kicad_pcb (KiCad board)
At the start: 2 copper layers, 159.9 x 99.9 mm, 4 parts

Commit message: Added rev 0.1 of logic debug
Signed-off-by: Matthew Nickson <mnickson@sidingsmedia.com>
Parts:
- added C1: 0.1uF, Capacitor_THT:C_Disc_D4.7mm_W2.5mm_P5.00mm, F.Cu at (65.1, 67.4)
- added C2: 0.1uF, Capacitor_THT:C_Disc_D4.7mm_W2.5mm_P5.00mm, F.Cu at (89.1, 89.9)
- added C3: 0.1uF, Capacitor_THT:C_Disc_D4.7mm_W2.5mm_P5.00mm, F.Cu at (75.1, 81.9)
- added D1: LED, LED_THT:LED_D3.0mm, F.Cu at (67.1, 50.9)
- added D2: LED, LED_THT:LED_D3.0mm, F.Cu at (59.1, 56.9)
- added D3: LED, LED_THT:LED_D3.0mm, F.Cu at (59.1, 61.9)
- added J1: DIN41612_02x16_AB, Connector_DIN:DIN41612_B2_2x16_Male_Horizontal_THT, F.Cu at (209.4, 75.9)
- added J2: USB_A, Connector_USB:USB_B_Lumberg_2411_02_Horizontal, F.Cu at (70.9, 85.2)
- added J3: Conn_01x16_Male, Connector_PinHeader_2.54mm:PinHeader_1x16_P2.54mm_Horizontal, F.Cu at (59.5, 132.9)
- added R1: 330R, Resistor_THT:R_Axial_DIN0207_L6.3mm_D2.5mm_P7.62mm_Horizontal, F.Cu at (79.9, 50.9)
- added R2: 4K7, Resistor_THT:R_Axial_DIN0207_L6.3mm_D2.5mm_P7.62mm_Horizontal, F.Cu at (95.1, 97.5)
- added R3: 4K7, Resistor_THT:R_Axial_DIN0207_L6.3mm_D2.5mm_P7.62mm_Horizontal, F.Cu at (85.9, 56.9)
- added R4: 330R, Resistor_THT:R_Axial_DIN0207_L6.3mm_D2.5mm_P7.62mm_Horizontal, F.Cu at (71.9, 56.9)
- added R5: 330R, Resistor_THT:R_Axial_DIN0207_L6.3mm_D2.5mm_P7.62mm_Horizontal, F.Cu at (71.9, 61.9)
- added R6: 4K7, Resistor_THT:R_Axial_DIN0207_L6.3mm_D2.5mm_P7.62mm_Horizontal, F.Cu at (85.9, 61.9)
- added SW1: SW_Push, Button_Switch_THT:SW_Tactile_SPST_Angled_PTS645Vx83-2LFS, F.Cu at (58.1, 71.9)
- added U1: MCP2221AxP, Package_DIP:DIP-14_W7.62mm, F.Cu at (85.9, 89.6)
Connections:
- MK1 pad : Net-(MK1-Pad1) -> (no net)
- MK2 pad : Net-(MK2-Pad1) -> (no net)
- MK3 pad : Net-(MK3-Pad1) -> (no net)
- MK4 pad : Net-(MK4-Pad1) -> (no net)
Routing:
- net /~{RESET}: track 0.00 -> 239.0 mm
- net /UART_RX0: track 0.00 -> 202.5 mm
- net /UART_TX0: track 0.00 -> 187.1 mm
- net /UART_RX2: track 0.00 -> 167.8 mm
- net /UART_TX2: track 0.00 -> 167.4 mm
- net /UART_RX1: track 0.00 -> 167.2 mm
- net /UART_TX1: track 0.00 -> 166.2 mm
- net /I2C_SDA: track 0.00 -> 150.4 mm
- net /SPI_~{CS_{2}}: track 0.00 -> 150.4 mm
- net /SPI_~{CS_{1}}: track 0.00 -> 150.4 mm
- net /SPI_SCLK: track 0.00 -> 150.4 mm
- net /SPI_MOSI: track 0.00 -> 150.4 mm
- net /SPI_MISO: track 0.00 -> 150.4 mm
- net /I2C_SCL: track 0.00 -> 150.4 mm
- net +5V: track 0.00 -> 69.2 mm
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- added copper zone on F.Cu, net +5V
- added copper zone on B.Cu, net GND
