File: logic-debug/logic-debug.kicad_sch (KiCad schematic)
At the start: 4 parts

Commit message: Added rev 0.1 of logic debug
Signed-off-by: Matthew Nickson <mnickson@sidingsmedia.com>
Parts:
- added C1, C2, C3: 0.1uF, Capacitor_THT:C_Disc_D4.7mm_W2.5mm_P5.00mm, symbol Device:C
- added D1, D2, D3: LED, LED_THT:LED_D3.0mm, symbol Device:LED
- added J1: DIN41612_02x16_AB, Connector_DIN:DIN41612_B2_2x16_Male_Horizontal_THT, symbol Connector:DIN41612_02x16_AB
- added J2: USB_A, symbol Connector:USB_A
- added J3: Conn_01x16_Male, Connector_PinHeader_2.54mm:PinHeader_1x16_P2.54mm_Horizontal, symbol Connector:Conn_01x16_Male
- added R1, R4, R5: 330R, Resistor_THT:R_Axial_DIN0207_L6.3mm_D2.5mm_P7.62mm_Horizontal, symbol Device:R
- added R2, R3, R6: 4K7, Resistor_THT:R_Axial_DIN0207_L6.3mm_D2.5mm_P7.62mm_Horizontal, symbol Device:R
- added SW1: SW_Push, Button_Switch_THT:SW_Tactile_SPST_Angled_PTS645Vx83-2LFS, symbol Switch:SW_Push
- added U1: MCP2221AxP, Package_DIP:DIP-14_W7.62mm, symbol Interface_USB:MCP2221AxP
Connections:
- new net: R6.2, U1.10 (SCL)
- new net: C3.1, U1.11 (VUSB)
- new net: R4.1, U1.2 (GP0)
- new net: R5.1, U1.3 (GP1)
- new net: R3.2, U1.9 (SDA)
- new net: D2.1 (K), R4.2
- new net: D1.1 (K), R1.2
- new net: D3.1 (K), R5.2
- new net +5V: C2.1, D1.2 (A), D2.2 (A), D3.2 (A), J1.b1 (Pin_b1), J1.b2 (Pin_b2), J3.15 (Pin_15), R2.1, R3.1, R6.1, U1.1 (VDD)
- new net D+: J2.3 (D+), U1.13 (D+)
- new net D-: J2.2 (D-), U1.12 (D-)
- new net GND: C1.2, C2.2, C3.2, J1.a7 (Pin_a7), J1.a8 (Pin_a8), J1.a9 (Pin_a9), J1.b7 (Pin_b7), J1.b8 (Pin_b8), J1.b9 (Pin_b9), J2.4 (GND), J2.5 (Shield), J3.16 (Pin_16), R1.1, SW1.1, U1.14 (VSS)
- new net I2C_SCL: J1.a15 (Pin_a15), J3.9 (Pin_9)
- new net I2C_SDA: J1.a16 (Pin_a16), J3.8 (Pin_8)
- new net SPI_MISO: J1.a12 (Pin_a12), J3.12 (Pin_12)
- new net SPI_MOSI: J1.a11 (Pin_a11), J3.13 (Pin_13)
- new net SPI_SCLK: J1.a10 (Pin_a10), J3.14 (Pin_14)
- new net SPI_~{CS_{1}}: J1.a13 (Pin_a13), J3.11 (Pin_11)
- new net SPI_~{CS_{2}}: J1.a14 (Pin_a14), J3.10 (Pin_10)
- new net UART_RX0: J1.b12 (Pin_b12), J3.6 (Pin_6), U1.6 (UTx)
- new net UART_RX1: J1.b14 (Pin_b14), J3.4 (Pin_4)
- new net UART_RX2: J1.b16 (Pin_b16), J3.2 (Pin_2)
- new net UART_TX0: J1.b11 (Pin_b11), J3.7 (Pin_7), U1.5 (URx)
- new net UART_TX1: J1.b13 (Pin_b13), J3.5 (Pin_5)
- new net UART_TX2: J1.b15 (Pin_b15), J3.3 (Pin_3)
- new net ~{RESET}: C1.1, J1.b10 (Pin_b10), J3.1 (Pin_1), R2.2, SW1.2, U1.4 (~{RST})
- no-connect marks 4 -> 17
Other:
- note added: "Backplane connector"
- note added: "Debug Header"
- note added: "Power LED"
- note added: "Rx and Tx LED"
- note added: "USB to UART"
